Commit message: lab7 finished

File: autlab7/urdf/kinect_sensor_jackal.urdf.xacro (robot description, xacro)
@@ -1,7 +1,7 @@
 <?xml version="1.0"?>
 <robot name="sensor_kinect" xmlns:xacro="http://ros.org/wiki/xacro">
-  <xacro:property name="cam_px" value="-0.0" />
+  <xacro:property name="cam_px" value="0.1" />
   <xacro:property name="cam_py" value="-0.0125" />
-  <xacro:property name="cam_pz" value="0.14" />
+  <xacro:property name="cam_pz" value="0.23" />
   <xacro:property name="cam_or" value="0" />
   <xacro:property name="cam_op" value="0" />
